File: BBoneSensorsCape.kicad_pcb (KiCad board)
At the start: 2 copper layers, 54.6 x 86.4 mm, 51 parts, among them J1 USB_B_Mini, J101 Conn_01x05, J2 Conn_01x04, J201 Conn_01x03, J3 Conn_01x05, J301 Conn_01x03, J4 Conn_01x08_MountingPin, P8 BeagleBone_Black_Header, P9 BeagleBone_Black_Header, SW101 SW_Push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

Commit message: Last cleanups, ready to manufacture
Signed-off-by: Alexis Jeandet <alexis.jeandet@member.fsf.org>
Parts:
- moved LOGO1 5.38 mm to (138.2, 105.6)
- moved LOGO2 3.51 mm to (126.1, 106.0)
Routing:
- net /RESET: track 66.8 -> 63.7 mm
- net GNDD: vias 125 -> 130
Other:
- board text added: "BBoneSensorsCape 1.0"
